Commit message: refresh

File: kobuki/kobuki_description/urdf/kobuki_gazebo.urdf.xacro (robot description, xacro)
@@ -42,5 +42,5 @@
 	      <visualize>true</visualize>
 	      <contact>
-	        <collision>base_footprint_fixed_joint_lump__base_collision</collision>
+	        <collision>base_footprint_collision_base_link</collision>
 	      </contact>
 	    </sensor>
@@ -160,5 +160,53 @@
       </sensor>
 	  </gazebo>
-	  <gazebo>
+       <gazebo>
+         <plugin name="differential_drive_controller" filename="libgazebo_ros_diff_drive.so">
+	    <alwaysOn>true</alwaysOn>
+	    <updateRate>20</updateRate>
+	    <leftJoint>wheel_left_joint</leftJoint>
+		<rightJoint>wheel_right_joint</rightJoint>
+	    <wheelSeparation>.230</wheelSeparation>
+	    <wheelDiameter>0.070</wheelDiameter>
+	    <torque>1.0</torque>
+	    <commandTopic>cmd_vel</commandTopic>
+	    <odometryTopic>odom</odometryTopic>
+	    <odometryFrame>odom</odometryFrame>
+	    <robotBaseFrame>base_footprint</robotBaseFrame>
+	    <publishWheelJointState>true</publishWheelJointState>
+	    <legacyMode>true</legacyMode>
+	  </plugin>
+	</gazebo>
+	<gazebo reference="laser_sensor_link">
+		<sensor type="gpu_ray" name="laser_sensor">
+			<pose>0 0 0 0 0 0</pose>
+			<visualize>false</visualize>
+			<update_rate>40</update_rate>
+			<ray>
+				<scan>
+					<horizontal>
+						<samples>720</samples>
+						<resolution>1</resolution>
+						<min_angle>-1.570796</min_angle>
+						<max_angle>1.570796</max_angle>
+					</horizontal>
+				</scan>
+				<range>
+					<min>0.10</min>
+					<max>30.0</max>
+					<resolution>0.01</resolution>
+				</range>
+				<noise>
+					<type>gaussian</type>
+					<mean>0.0</mean>
+					<stddev>0.01</stddev>
+				</noise>
+			</ray>
+			<plugin name="gazebo_ros_head_hokuyo_controller" filename="libgazebo_ros_gpu_laser.so">
+				<topicName>/kobuki/laser/scan</topicName>
+				<frameName>laser_sensor_link</frameName>
+			</plugin>
+		</sensor>
+	</gazebo>
+          <!--gazebo>
 	    <plugin name="kobuki_controller" filename="libgazebo_ros_kobuki.so">
 	      <publish_tf>1</publish_tf>
@@ -176,5 +224,5 @@
         <imu_name>imu</imu_name>
 	    </plugin>
-	  </gazebo>
+	  </gazebo-->
   </xacro:macro>
 </robot>
